File: KiCAD/YM2151.sch (KiCad schematic (older format))
At the start: 32 parts, among them J1 AudioJack3_Ground, P1 Power, P2 Analog, P3 Digital, P4 Digital, P5 CONN_01X01, P6 CONN_01X01, P7 CONN_01X01, P8 CONN_01X01, U1 YM2151, U2 YM3012, U3 LMC6484, U4 74LS04, U5 74LS00, U6 C64-Exp-Port

Commit message: microcontroller added
Parts:
- removed C4, C5: 4.7u, Capacitor_THT:CP_Radial_D5.0mm_P2.50mm, symbol Device:CP
- removed NT1: Net-Tie_2, NetTie:NetTie-2_SMD_Pad2.0mm, symbol Device:Net-Tie_2
- removed P5, P6, P7, P8: CONN_01X01, Socket_Arduino_Uno:Arduino_1pin, symbol YM2151-rescue:CONN_01X01
- added C4, C5: 4.7u, Capacitor_SMD:C_0805_2012Metric, symbol Device:C
- added H2, H3, H4, H5: MountingHole, MountingHole:MountingHole_3.2mm_M3, symbol Mechanical:MountingHole
- C1, C10, C11, C6: footprint Capacitor_THT:CP_Radial_D5.0mm_P2.50mm -> Capacitor_SMD:C_0805_2012Metric
- C2, C3: footprint Capacitor_THT:C_Disc_D4.3mm_W1.9mm_P5.00mm -> Capacitor_SMD:C_0805_2012Metric
- C7, C8, C9: footprint Capacitor_THT:C_Disc_D3.0mm_W1.6mm_P2.50mm -> Capacitor_SMD:C_0805_2012Metric
- R1, R2: footprint Resistors_THT:R_Axial_DIN0204_L3.6mm_D1.6mm_P7.62mm_Horizontal -> Resistor_SMD:R_0805_2012Metric
- R5: footprint Resistor_THT:R_Axial_DIN0204_L3.6mm_D1.6mm_P7.62mm_Horizontal -> Resistor_SMD:R_0805_2012Metric
- U3: footprint Housings_DIP:DIP-14_W7.62mm_Socket -> Package_SO:SOIC-14_3.9x8.7mm_P1.27mm
Connections:
- net GNDA is gone; now on net GNDD: C1.2, C2.2, C3.2, J1.S, U2.16 (A-GND), U2.8 (A-GND), U3.11 (V-), U3.11 (V-), U3.11 (V-), U3.11 (V-)
- net ~CS is gone; now on net PHI2: P2.1 (P1)
- net ~RD is gone; now on net ~IO1: P3.8 (P8)
- net ~WR is gone; now on net R~W: P3.7 (P7)
- net A1: now also P2.3 (P3)
- net GNDD: no longer U4.13, U5.12, U5.13
- net PHI2: now also U5.13; no longer U5.5
- net A7: now reaches P2.2 (P2)
- net A7: now also U5.5, U6.R (A7)
- net at U1.7 (~CS): now also U5.11; no longer U5.6
- net at U3.13 (-), U3.14: now also C5.2
- net at U3.8, U3.9 (-): now also C4.2
- net at R1.2: now also C4.1
- net at R2.2: now also C5.1
- net ~IO1: now reaches U6.7 (/I/O1)
- net ~IO1: now also U4.5
- net at U4.12: now also U5.12
- net ~IO2: no longer names the net of U6.10 (/I/O2)
- net ~IO2: no longer U4.5
- new net: U4.13, U5.6
- no-connect marks 44 -> 36
Other:
- note added: "unused gates"
- note removed: "Holes"
- moved on the sheet: O1, U4A, U4B, U4C, U4D, U4E, U4F, U5B, U5C, U5D

Commit message: board routed
Parts:
- removed C1: 10u, Capacitor_SMD:C_0805_2012Metric, symbol Device:CP
- removed C10, C11, C6: 4.7u, Capacitor_SMD:C_0805_2012Metric, symbol Device:CP
- removed P1: Power, Socket_Arduino_Uno:Socket_Strip_Arduino_1x08, symbol YM2151-rescue:CONN_01X08
- removed P2: Analog, Socket_Arduino_Uno:Socket_Strip_Arduino_1x06, symbol YM2151-rescue:CONN_01X06
- removed P3: Digital, Socket_Arduino_Uno:Socket_Strip_Arduino_1x10, symbol YM2151-rescue:CONN_01X10
- removed P4: Digital, Socket_Arduino_Uno:Socket_Strip_Arduino_1x08, symbol YM2151-rescue:CONN_01X08
- added C1: 4.7n/250V, Capacitor_SMD:C_0805_2012Metric, symbol Device:C
- added C12, C13, C14, C23, C24, C27: 10u, Capacitor_SMD:C_0805_2012Metric, symbol Device:C
- added C15: 1uF, Capacitor_SMD:C_0805_2012Metric, symbol Device:C
- added C16, C17, C22, C26: 1u, Capacitor_SMD:C_0805_2012Metric, symbol Device:C
- added C18, C19, C20, C21, C25, C7: 100n, Capacitor_SMD:C_0805_2012Metric, symbol Device:C
- added C5, C6: 15p, Capacitor_SMD:C_0805_2012Metric, symbol Device:C
- added D1: LED, LED_SMD:LED_0805_2012Metric, symbol Device:LED
- added FB1, FB2: Ferrite_Bead, Inductor_SMD:L_1206_3216Metric, symbol Device:Ferrite_Bead
- added J10, J11, J12, J13, J14, J15, J16, J5, J6, J7, J8, J9: IO, Connector_PinHeader_2.54mm:PinHeader_1x01_P2.54mm_Vertical, symbol Connector:Conn_01x01_Male
- added J17: +5V, Connector_PinHeader_2.54mm:PinHeader_1x01_P2.54mm_Vertical, symbol Connector:Conn_01x01_Male
- added J18: GND, Connector_PinHeader_2.54mm:PinHeader_1x01_P2.54mm_Vertical, symbol Connector:Conn_01x01_Male
- added J19: +3.3V, Connector_PinHeader_2.54mm:PinHeader_1x01_P2.54mm_Vertical, symbol Connector:Conn_01x01_Male
- added J2: 690-005-299-043, KiCAD:USB_Mini_B_Female_690-005-299-043, symbol dk_USB-DVI-HDMI-Connectors:690-005-299-043
- added J3: TXO, Connector_PinHeader_2.54mm:PinHeader_1x01_P2.54mm_Vertical, symbol Connector:Conn_01x01_Male
- added J4: TXI, Connector_PinHeader_2.54mm:PinHeader_1x01_P2.54mm_Vertical, symbol Connector:Conn_01x01_Male
- added P1: SWD, swd:swd, symbol swd:SWD
- added R10, R11, R4, R9: 10k, Resistor_SMD:R_0805_2012Metric, symbol Device:R
- added R12, R13, R14, R15, R6, R7: 33, Resistor_SMD:R_0805_2012Metric, symbol Device:R
- added R5: 1M, Resistor_SMD:R_0805_2012Metric, symbol Device:R
- added R8: 1k, Resistor_SMD:R_0805_2012Metric, symbol Device:R
- added RN1, RN2: 100k, Resistor_SMD:R_Array_Convex_8x0602, symbol Device:R_Pack08
- added U10: MCP1700-3302E_SOT23, Package_TO_SOT_SMD:SOT-23, symbol Regulator_Linear:MCP1700-3302E_SOT23
- added U7, U9: SN74AVC8T245PW, Package_SO:TSSOP-24_4.4x7.8mm_P0.65mm, symbol Logic_LevelTranslator:SN74AVC8T245PW
- added U8: ATSAMD21G18A-AU, ATSAMD21G18A-AU:QFP50P900X900X120-48N, symbol ATSAMD21G18A-AU:ATSAMD21G18A-AU
- added Y1: Crystal, Crystal:Crystal_SMD_3215-2Pin_3.2x1.5mm, symbol Device:Crystal
- C10: renamed from C4; value 4.7u -> 10u
- C11: renamed from C5; value 4.7u -> 10u
- U4: renamed from U1; footprint Housings_DIP:DIP-24_W15.24mm_Socket -> Package_DIP:DIP-24_W15.24mm_LongPads
- U5: renamed from U2; footprint Housings_DIP:DIP-16_W7.62mm_Socket -> Package_DIP:DIP-16_W7.62mm_Socket_LongPads
- renumbered C7 to C2, C8 to C3, C9 to C4, C2 to C8, C3 to C9, R5 to R1, R1 to R2, R2 to R3, U4 to U1, U5 to U2, U6 to U3, U3 to U6
Connections:
- net A0: now also RN2.13 (R4.2), U9.17 (B5)
- net A1: now also RN2.14 (R3.2), U9.16 (B6)
- net A7: now also RN2.15 (R2.2), U9.15 (B7)
- net D0: now also RN1.9 (R8.2), U7.21 (B1)
- net D1: now also RN1.10 (R7.2), U7.20 (B2)
- net D2: now also RN1.11 (R6.2), U7.19 (B3)
- net D3: now also RN1.12 (R5.2), U7.18 (B4)
- net D4: now also RN1.13 (R4.2), U7.17 (B5)
- net D5: now also RN1.14 (R3.2), U7.16 (B6)
- net D6: now also RN1.15 (R2.2), U7.15 (B7)
- net D7: now also RN1.16 (R1.2), U7.14 (B8)
- net PHI2: now also RN2.12 (R5.2), U9.18 (B4)
- net R~W: now also RN2.10 (R7.2), U9.20 (B2)
- net VCC: now also C12.1, C13.1, C14.1, C16.1, FB1.1, FB2.1, J17.1 (Pin_1), J2.1, P1.5 (5V-Supply), U10.3 (VI), U7.23 (VCCB), U7.24 (VCCB), U9.23 (VCCB); no longer U5.1 (Vcc), U6.4 (V+), U6.4 (V+), U6.4 (V+), U6.4 (V+)
- net ~IC: now also RN2.11 (R6.2), U9.19 (B3)
- net ~IO1: now also RN2.9 (R8.2), U9.21 (B1)
- net at U4.19 (SH2): now also R15.2; no longer U5.5 (SH2)
- net at U4.20 (SH1): now also R14.2; no longer U5.6 (SH1)
- net at U4.21 (SO): now also R13.2; no longer U5.4 (DATA)
- net at U4.23 (phi1): now also R12.2; no longer U5.2 (phi1)
- net at U5.15 (RB(BIAS)), U6.3 (+): now also C24.1
- net GNDD renamed GND
- net GND: now also C1.2, C12.2, C13.2, C14.2, C15.2, C16.2, C17.2, C18.2, C19.2, C20.2, C21.2, C22.2, C23.2, C24.2, C25.2, C26.2, C27.2, C5.2, C6.2, C7.2, D1.1 (K), J18.1 (Pin_1), J2.5, P1.3 (GND), R10.2, R11.1, R4.1, R5.1, RN1.1 (R1.1), RN1.2 (R2.1), RN1.3 (R3.1), RN1.4 (R4.1), RN1.5 (R5.1), RN1.6 (R6.1), RN1.7 (R7.1), RN1.8 (R8.1), RN2.1 (R1.1), RN2.2 (R2.1), RN2.3 (R3.1), RN2.4 (R4.1), RN2.5 (R5.1), RN2.6 (R6.1), RN2.7 (R7.1), RN2.8 (R8.1), U10.1 (GND), U7.11 (GND), U7.12 (GND), U7.13 (GND), U7.22 (~OE), U8.18 (GND1), U8.35 (GND2), U8.42 (GND3), U8.5 (GNDANA), U9.11 (GND), U9.12 (GND), U9.13 (GND), U9.22 (~OE)
- new net: C22.1, C23.1, C7.1, FB1.2, U5.1 (Vcc)
- new net: R12.1, U5.2 (phi1)
- new net: R13.1, U5.4 (DATA)
- new net: R15.1, U5.5 (SH2)
- new net: R14.1, U5.6 (SH1)
- new net: C25.1, C26.1, C27.1, FB2.2, U6.4 (V+), U6.4 (V+), U6.4 (V+), U6.4 (V+)
- new net: C15.1, U8.43 (VDDCORE)
- new net: R6.1, U8.33 (PA24)
- new net: R7.1, U8.34 (PA25)
- new net: U7.10 (A8), U8.14 (PA09)
- new net: R4.2, U7.2 (DIR), U8.21 (PA12)
- new net: U7.3 (A1), U8.3 (PA02)
- new net: U7.4 (A2), U8.4 (PA03)
- new net: U7.5 (A3), U8.9 (PA04)
- new net: U7.6 (A4), U8.10 (PA05)
- new net: U7.7 (A5), U8.11 (PA06)
- new net: U7.8 (A6), U8.12 (PA07)
- new net: U7.9 (A7), U8.13 (PA08)
- new net: R10.1, U9.10 (A8)
- new net: RN2.16 (R1.2), U9.14 (B8)
- new net: R11.2, U8.47 (PB02), U9.2 (DIR)
- new net: U8.48 (PB03), U9.3 (A1)
- new net: U8.7 (PB08), U9.4 (A2)
- new net: U8.8 (PB09), U9.5 (A3)
- new net: U8.19 (PB10), U9.6 (A4)
- new net: U8.20 (PB11), U9.7 (A5)
- new net: U8.37 (PB22), U9.8 (A6)
- new net: U8.38 (PB23), U9.9 (A7)
- new net: C1.1, J2.SH, R5.2
- new net: D1.2 (A), R8.1
- new net: R8.2, U8.26 (PA17)
- new net: C5.1, U8.1 (PA00), Y1.1
- new net: C6.1, U8.2 (PA01), Y1.2
- new net: J3.1 (Pin_1), U8.15 (PA10)
- new net: J4.1 (Pin_1), U8.16 (PA11)
- new net: J5.1 (Pin_1), U8.22 (PA13)
- new net: J6.1 (Pin_1), U8.23 (PA14)
- new net: J7.1 (Pin_1), U8.24 (PA15)
- new net: J8.1 (Pin_1), U8.25 (PA16)
- new net: J9.1 (Pin_1), U8.27 (PA18)
- new net: J10.1 (Pin_1), U8.28 (PA19)
- new net: J11.1 (Pin_1), U8.29 (PA20)
- new net: J12.1 (Pin_1), U8.30 (PA21)
- new net: J13.1 (Pin_1), U8.31 (PA22)
- new net: J14.1 (Pin_1), U8.32 (PA23)
- new net: J15.1 (Pin_1), U8.39 (PA27)
- new net: J16.1 (Pin_1), U8.41 (PA28)
- new net +3V3: C17.1, C18.1, C19.1, C20.1, C21.1, J19.1 (Pin_1), P1.1 (VTref), R9.1, U10.2 (VO), U7.1 (VCCA), U8.17 (VDDIO1), U8.36 (VDDIO2), U8.44 (VDDIN), U8.6 (VDDANA), U9.1 (VCCA), U9.24 (VCCB)
- new net D+: J2.3, R7.2
- new net D-: J2.2, R6.2
- new net RESET: P1.10 (nRESET), R9.2, U8.40 (~RESETN~)
- new net SWCLK: P1.4 (SWCLK/TCK), U8.45 (PA30)
- new net SWDIO: P1.2 (SWDIO/TMS), U8.46 (PA31)
- no-connect marks 36 -> 33
Other:
- note added: "USB shield\nEMI termination"
- note removed: "1"
- note removed: "Shield for Arduino that uses\nthe same pin disposition\nlike "Uno" board Rev 3."
- moved on the sheet: H2, H3, H4, H5, U1A, U1D, U1E

Commit message: REV B
Connections:
- net +3V3: no longer U9.24 (VCCB)
- net VCC: now also U9.24 (VCCB)
Changed lines of the file:
@@
 	3350 7200 3350 7050
 Wire Wire Line
-	9150 7700 9150 7550
-Wire Wire Line
-	8950 7700 8950 7650
-Wire Wire Line
-	9050 7700 9050 7650
-Wire Wire Line
-	9050 7650 8950 7650
-Connection ~ 8950 7650
-Wire Wire Line
-	8950 7650 8950 7550
+	9150 7700 9150 7650
 Wire Wire Line
 	7900 10650 8500 10650
@@
 NoConn ~ 12200 2850
 NoConn ~ 10400 2850
+Wire Wire Line
+	8950 7550 8950 7700
+Wire Wire Line
+	9150 7650 9050 7650
+Wire Wire Line
+	9050 7650 9050 7700
 Wire Bus Line
 	950  3200 3450 3200
@@
 Wire Bus Line
 	1150 1150 1150 3100
+Connection ~ 9150 7650
+Wire Wire Line
+	9150 7650 9150 7550
 $EndSCHEMATC
